File: Flight_Controller/Power.kicad_sch (KiCad schematic)
At the start: 0 parts

Commit message: Schem V1 Done!
Parts:
- added C10: 33nF, PCM_JLCPCB:C_0603, symbol PCM_JLCPCB-Capacitors:0603,33nF
- added C11, C7: 100nF, PCM_JLCPCB:C_0603, symbol PCM_JLCPCB-Capacitors:0603,100nF
- added C12: 6.8pF, PCM_JLCPCB:C_0603, symbol PCM_JLCPCB-Capacitors:0603,6.8pF
- added C13: 47uF, PCM_JLCPCB:C_0805, symbol PCM_JLCPCB-Capacitors:0805,47uF
- added C14, C15: 1uF, PCM_JLCPCB:C_0603, symbol PCM_JLCPCB-Capacitors:0603,1uF
- added C5: 10uF, PCM_JLCPCB:C_0603, symbol PCM_JLCPCB-Capacitors:0603,10uF
- added J1: ESC->FC DSHOT and Telem, symbol Connector:Conn_01x08_Socket
- added J2: ELRS Reciever, symbol Connector:Conn_01x04_Socket
- added J3: VTX, symbol Connector:Conn_01x06_Socket
- added J4: Conn_01x03_Socket, symbol Connector:Conn_01x03_Socket
- added J5: USB_C_Receptacle_USB2.0_16P, symbol Connector:USB_C_Receptacle_USB2.0_16P
- added L1: 12uH, symbol Device:L
- added R10, R9: 5.1kΩ, PCM_JLCPCB:R_0603, symbol PCM_JLCPCB-Resistors:0603,5.1kΩ
- added R7: 52.3K, symbol Device:R
- added R8: 10kΩ, PCM_JLCPCB:R_0603, symbol PCM_JLCPCB-Resistors:0603,10kΩ
- added U3: TLV75533PDBV, Package_TO_SOT_SMD:SOT-23-5, symbol Regulator_Linear:TLV75533PDBV
- added U5: TPS62932, Package_TO_SOT_SMD:SOT-583-8, symbol Regulator_Switching:TPS62932
- added U6: TPD2EUSB30ADRTR, Flight_Controller:DRT3-L, symbol Flight_Controller:TPD2EUSB30ADRTR
Connections:
- new net: C10.1, U5.7 (SS)
- new net +3V3: C15.1, U3.5 (OUT)
- new net +5V: C12.1, C13.1, C14.1, J2.1 (Pin_1), J3.1 (Pin_1), J4.1 (Pin_1), L1.2, R7.1, U3.1 (IN), U3.3 (EN)
- new net +5V_USB: J5.A4 (VBUS), J5.A9 (VBUS), J5.B4 (VBUS), J5.B9 (VBUS)
- new net +BATT: C5.1, C7.1, U5.3 (VIN)
- new net ADC_CURR: J1.1 (Pin_1)
- new net BST: C11.1, U5.6 (BST)
- new net CC1: J5.A5 (CC1), R9.2
- new net CC2: J5.B5 (CC2), R10.2
- new net D+: J5.A6 (D+), J5.B6 (D+), U6.1 (D+)
- new net D-: J5.A7 (D-), J5.B7 (D-), U6.2 (D-)
- new net ELRS_RX: J2.2 (Pin_2)
- new net ELRS_TX: J2.3 (Pin_3)
- new net FB: C12.2, R7.2, R8.1, U5.8 (FB)
- new net GND: C10.2, C13.2, C14.2, C15.2, C5.2, C7.2, J1.7 (Pin_7), J1.8 (Pin_8), J2.4 (Pin_4), J3.6 (Pin_6), J4.3 (Pin_3), J5.A1 (GND), J5.A12 (GND), J5.B1 (GND), J5.B12 (GND), J5.SH (SHIELD), R10.1, R8.2, R9.1, U3.2 (GND), U5.4 (GND), U6.3 (GND)
- new net M1_DSHOT: J1.3 (Pin_3)
- new net M2_DSHOT: J1.4 (Pin_4)
- new net M3_DSHOT: J1.5 (Pin_5)
- new net M4_DSHOT: J1.6 (Pin_6)
- new net SW: C11.2, L1.1, U5.5 (SW)
- new net TELEM_RX: J1.2 (Pin_2)
- new net VIDEO_IN: J4.2 (Pin_2)
- new net VIDEO_OUT: J3.4 (Pin_4), J3.5 (Pin_5)
- new net VTX_RX: J3.2 (Pin_2)
- new net VTX_TX: J3.3 (Pin_3)
- no-connect marks 0 -> 4
