File: Flight_Controller/architecture.kicad_sch (KiCad schematic)
At the start: 0 parts

Commit message: Schem V1 Done!
Other:
- sheet MCU renamed MCU/Connectors
- sheet Peripherals renamed Peripherals/Power
- removed sheet Power
- sheet MCU/Connectors ports: added +3V3, +5V, +BATT, BB_SPI_CS, IMU_INT, IMU_SPI_CS, IMU_SPI_SCK, IMU_SPI_SDI, IMU_SPI_SDO, LPS_INT, LPS_SPI_CS, OSD_LOS, OSD_SPI_CS, OSD_VS, SPI_CLK, SPI_SDI, SPI_SDO, VIDEO_IN, VIDEO_OUT; removed none
- sheet Peripherals/Power ports: added +3V3, +5V, +BATT, BB_SPI_CS, BMI_SPI_CS, IMU_INT, IMU_SPI_SCK, IMU_SPI_SDI, IMU_SPI_SDO, LPS_INT, LPS_SPI_CS, OSD_LOS, OSD_SPI_CS, OSD_VS, SPI_SCK, SPI_SDI, SPI_SDO, VIDEO_IN, VIDEO_OUT; removed none
