File: Flight_Controller/MCU.kicad_sch (KiCad schematic)
At the start: 37 parts, among them J10 USB_C_Receptacle_USB2.0_16P, J11 Conn_ARM_SWD_TagConnect_TC203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, J13 SM06B-GHS-TB, J14 VTX, J6 ESC->FC DSHOT and Telem, J7 ELRS Reciever, J9 Camera, SW1 SW_Push, U1 STM32H743VITx, U7 TPD2EUSB30ADRTR

Commit message: Initial Layout Done
Connections:
- net +BATT: now also J6.1 (Pin_1); no longer J6.7 (Pin_7)
- net ADC_CURR: now also J6.7 (Pin_7); no longer J6.1 (Pin_1)
- net MCU_LED: now reaches D1.1, R9.2
- net USB_LED: now reaches D2.1, R10.1
Other:
- moved on the sheet: R10

Commit message: Updated Connector Standard
Parts:
- removed D1: Red, PCM_JLCPCB:D_0603, symbol PCM_JLCPCB-Diodes:LED,0603,Red
- removed R9: 150Ω, PCM_JLCPCB:R_0603, symbol PCM_JLCPCB-Resistors:0603,150Ω
- added D8: Red, PCM_JLCPCB:D_0603, symbol PCM_JLCPCB-Diodes:LED,0603,Red
- added R19: 150Ω, PCM_JLCPCB:R_0603, symbol PCM_JLCPCB-Resistors:0603,150Ω
Connections:
- net +BATT: now also J6.8 (Pin_8); no longer J6.1 (Pin_1)
- net ADC_CURR: now also J6.1 (Pin_1); no longer J6.7 (Pin_7)
- net GND: now also J6.7 (Pin_7), R19.1; no longer J6.8 (Pin_8)
- net PB10: now reaches U1.46 (PB10)
- net PB10: now also D8.2
- new net 3V3_LED: D8.1, R19.2
- no-connect marks 52 -> 51

Commit message: Added 9V Buck, GPS + Mag, Digital VTX
Parts:
- removed J14: VTX, Connector_JST:JST_GH_SM06B-GHS-TB_1x06-1MP_P1.25mm_Horizontal, symbol Connector_Generic:Conn_01x06
- removed R14: 10kΩ, PCM_JLCPCB:R_0603, symbol PCM_JLCPCB-Resistors:0603,10kΩ
- added J1: Analog VTX, symbol Connector_Generic:Conn_01x05
- added J2: Digital VTX, symbol Connector_Generic:Conn_01x06
- added J3: GPS+Mag, symbol Connector_Generic:Conn_01x06
Connections:
- net RST_SW is gone; now on net GND: SW1.1
- net +5V: now also J3.3 (Pin_3)
- net +BATT: now also J6.1 (Pin_1); no longer J6.8 (Pin_8)
- net ADC_CURR: now also J6.3 (Pin_3); no longer J6.1 (Pin_1)
- net ELRS_RX: now also J7.3 (Pin_3); no longer J7.2 (Pin_2)
- net ELRS_TX: now also J7.4 (Pin_4); no longer J7.3 (Pin_3)
- net GND: now also J6.2 (Pin_2), J7.2 (Pin_2), J9.2 (Pin_2), J1.2 (Pin_2), J2.2 (Pin_2), J2.5 (Pin_5), J3.4 (Pin_4); no longer J6.7 (Pin_7), J7.4 (Pin_4), J9.3 (Pin_3)
- net M1_DSHOT: now also J6.5 (Pin_5); no longer J6.3 (Pin_3)
- net M2_DSHOT: now also J6.6 (Pin_6); no longer J6.4 (Pin_4)
- net M3_DSHOT: now also J6.7 (Pin_7); no longer J6.5 (Pin_5)
- net M4_DSHOT: now also J6.8 (Pin_8); no longer J6.6 (Pin_6)
- net TELEM_RX: now also J6.4 (Pin_4); no longer J6.2 (Pin_2)
- net VIDEO_IN: now also J9.3 (Pin_3); no longer J9.2 (Pin_2)
- net VIDEO_OUT: now also J1.3 (Pin_3)
- net VTX_RX: now also J1.4 (Pin_4)
- net VTX_TX: now also J1.5 (Pin_5)
- new net +9V: J1.1 (Pin_1), J2.1 (Pin_1)
- new net DVTX_RX: J2.4 (Pin_4)
- new net DVTX_TX: J2.3 (Pin_3)
- new net GPS_RX: J3.5 (Pin_5)
- new net GPS_TX: J3.6 (Pin_6)
- new net SBUS: J2.6 (Pin_6)
- new net SCL: J3.2 (Pin_2)
- new net SDA: J3.1 (Pin_1)
Other:
- moved on the sheet: J9

Commit message: Updated Footprints
Parts:
- removed J6: ESC->FC DSHOT and Telem, Connector_JST:JST_GH_SM08B-GHS-TB_1x08-1MP_P1.25mm_Horizontal, symbol Connector:Conn_01x08_Socket
- added J4: ESC Connector, Connector_JST:JST_SH_SM10B-SRSS-TB_1x10-1MP_P1.00mm_Horizontal, symbol Connector_Generic:Conn_01x10
- J1: footprint (none) -> Connector_JST:JST_SH_SM05B-SRSS-TB_1x05-1MP_P1.00mm_Horizontal
- J2, J3: footprint (none) -> Connector_JST:JST_SH_SM06B-SRSS-TB_1x06-1MP_P1.00mm_Horizontal
- J7: footprint Connector_JST:JST_GH_SM04B-GHS-TB_1x04-1MP_P1.25mm_Horizontal -> Connector_JST:JST_SH_SM04B-SRSS-TB_1x04-1MP_P1.00mm_Horizontal
- J9: footprint Connector_JST:JST_GH_SM03B-GHS-TB_1x03-1MP_P1.25mm_Horizontal -> Connector_JST:JST_SH_SM03B-SRSS-TB_1x03-1MP_P1.00mm_Horizontal
- SW1: footprint Resistor_SMD:R_0805_2012Metric -> Flight_Controller:SW_TS-1088-AR02016
Connections:
- net SCL is gone; now on net Mag_SCL: J3.2 (Pin_2)
- net SDA is gone; now on net Mag_SDA: J3.1 (Pin_1)
- net +BATT: now also J4.1 (Pin_1)
- net ADC_CURR: now also J4.3 (Pin_3)
- net DVTX_RX: now also U1.37 (PE7)
- net DVTX_TX: now also U1.38 (PE8)
- net GND: now also J4.2 (Pin_2)
- net GPS_RX: now also U1.92 (PB6)
- net GPS_TX: now also U1.91 (PB5)
- net M1_DSHOT: now also J4.5 (Pin_5)
- net M2_DSHOT: now also J4.6 (Pin_6)
- net M3_DSHOT: now also J4.7 (Pin_7)
- net M4_DSHOT: now also J4.8 (Pin_8)
- net SBUS: now also U1.64 (PC7)
- net TELEM_RX: now also J4.4 (Pin_4)
- net Mag_SCL: now reaches U1.59 (PD12)
- net Mag_SDA: now reaches U1.60 (PD13)
- net M5_DSHOT: now reaches U1.61 (PD14)
- net M5_DSHOT: now also J4.9 (Pin_9)
- net M6_DSHOT: now reaches U1.62 (PD15)
- net M6_DSHOT: now also J4.10 (Pin_10)
- no-connect marks 51 -> 42
Other:
- note added: "UART_4"
- note added: "UART_5"
- note added: "UART_7"
- note added: "USART_2"
- note added: "USART_3"
- note added: "USART_6"
