File: Flight_Controller/.history/Flight_Controller.kicad_pcb (KiCad board)
At the start: 4 copper layers, 38 x 68 mm, 94 parts, among them IC1 AT7456E, J1 Analog VTX, J10 USB_C_Receptacle_USB2.0_16P, J11 Conn_ARM_SWD_TagConnect_TC203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, J13 SM06B-GHS-TB, J2 Digital VTX, J3 GPS+Mag, J4 ESC Connector, J7 ELRS Reciever, J9 Camera, SW1 SW_Push, U1 STM32H743VITx, U2 BMI270, U3 TLV75533PDBV, U4 W25Q128JVSIQ TR, U6 LMR51625XDDCR, U7 TPD2EUSB30ADRTR, U8 LMR51625XDDCR, Y2 ABM3-27.000MHZ-D2Y-T

Commit message: Routing Done!
Parts:
- removed J1: Analog VTX, Connector_JST:JST_SH_SM05B-SRSS-TB_1x05-1MP_P1.00mm_Horizontal
- removed R14: 10kΩ, PCM_JLCPCB:R_0603
- removed R8: 20kΩ, PCM_JLCPCB:R_0603
- added G***: LOGO, LOGO, B.Cu at (121.7, 91.9)
- added G***: LOGO, LOGO, B.Cu at (104.8, 90.7)
- added G***: LOGO, LOGO, B.Cu at (114.7, 72.3)
- added R20: 10kΩ, PCM_JLCPCB:R_0603, F.Cu at (125.4, 104.7)
- added TP1: TestPoint, TestPoint:TestPoint_Pad_D1.0mm, F.Cu at (111.8, 55.1)
- added TP10: TestPoint, TestPoint:TestPoint_Pad_D1.0mm, B.Cu at (104.5, 52.7)
- added TP13: TestPoint, TestPoint:TestPoint_Pad_D1.0mm, B.Cu at (109.4, 52.7)
- added TP16: TestPoint, TestPoint:TestPoint_Pad_D1.0mm, B.Cu at (104.5, 49.1)
- added TP17: TestPoint, TestPoint:TestPoint_Pad_D1.0mm, B.Cu at (116.5, 49.1)
- added TP18: TestPoint, TestPoint:TestPoint_Pad_D1.0mm, B.Cu at (107.0, 49.1)
- added TP19: TestPoint, TestPoint:TestPoint_Pad_D1.0mm, B.Cu at (109.4, 49.1)
- added TP2: TestPoint, TestPoint:TestPoint_Pad_D1.0mm, F.Cu at (108.4, 55.1)
- added TP20: TestPoint, TestPoint:TestPoint_Pad_D1.0mm, B.Cu at (111.8, 49.1)
- added TP21: TestPoint, TestPoint:TestPoint_Pad_D1.0mm, B.Cu at (114.2, 49.1)
- added TP22: TestPoint, TestPoint:TestPoint_Pad_D1.0mm, B.Cu at (114.2, 52.7)
- added TP23: TestPoint, TestPoint:TestPoint_Pad_D1.0mm, B.Cu at (111.8, 52.7)
- added TP24: TestPoint, TestPoint:TestPoint_Pad_D1.0mm, B.Cu at (118.9, 49.1)
- added TP25: TestPoint, TestPoint:TestPoint_Pad_D1.0mm, B.Cu at (121.3, 49.1)
- added TP26: TestPoint, TestPoint:TestPoint_Pad_D1.0mm, B.Cu at (121.3, 52.7)
- added TP3: TestPoint, TestPoint:TestPoint_Pad_D1.0mm, F.Cu at (115.3, 55.1)
- added TP4: TestPoint, TestPoint:TestPoint_Pad_D1.0mm, F.Cu at (122.3, 55.1)
- added TP5: TestPoint, TestPoint:TestPoint_Pad_D1.0mm, F.Cu at (104.7, 55.1)
- added TP6: TestPoint, TestPoint:TestPoint_Pad_D1.0mm, F.Cu at (113.3, 58.0)
- added TP7: TestPoint, TestPoint:TestPoint_Pad_D1.0mm, B.Cu at (118.9, 52.7)
- added TP8: TestPoint, TestPoint:TestPoint_Pad_D1.0mm, B.Cu at (116.5, 52.7)
- added TP9: TestPoint, TestPoint:TestPoint_Pad_D1.0mm, B.Cu at (107.0, 52.7)
- R1: value 1kΩ -> 53.6K
- R3: value 1kΩ -> 10.2K
- R7: value 100kΩ -> 9.76K
- moved C27 49.4 mm to (125.5, 103.1)
- moved SW1 49.4 mm to (126.8, 100.3)
- moved R3 43.3 mm to (105.1, 102.0), turned to 180 degrees
- moved R1 42.3 mm to (105.1, 103.4)
- moved J2 9.97 mm to (129.5, 92.1)
- moved R7 6.88 mm to (112.0, 103.4), turned to 180 degrees
- moved NT2 4.36 mm to (114.1, 68.8), turned to 180 degrees
- moved NT1 3.79 mm to (109.0, 63.2)
- moved NT4 2.44 mm to (119.0, 67.1)
- moved NT3 1.02 mm to (107.4, 63.3)
- moved C30 0.94 mm to (118.4, 67.9)
- moved C29 0.13 mm to (118.5, 89.2)
- moved C16 0.12 mm to (119.8, 89.2)
- moved C28 0.09 mm to (123.3, 74.8)
Connections:
- A1 pad 2: /MCU/Connectors/SPI_SCK -> /MCU/Connectors/I2C_SCL1
- A1 pad 4: /MCU/Connectors/SPI_SDI -> /MCU/Connectors/I2C_SDA1
- A1 pad 5: /MCU/Connectors/SPI_SDO -> unconnected-(A1-SDO/SA0-Pad5)
- A1 pad 6: /MCU/Connectors/LPS_SPI_CS -> unconnected-(A1-CS-Pad6)
- IC1 pad 10: /MCU/Connectors/SPI_SCK -> /MCU/Connectors/OSD_SPI_SCK
- IC1 pad 11: /MCU/Connectors/SPI_SDO -> /MCU/Connectors/OSD_SPI_SDO
- IC1 pad 12: /MCU/Connectors/OSD_LOS -> unconnected-(IC1-LOS-Pad12)
- IC1 pad 17: /MCU/Connectors/OSD_VS -> unconnected-(IC1-~{VSYNC}-Pad17)
- IC1 pad 9: /MCU/Connectors/SPI_SDI -> /MCU/Connectors/OSD_SPI_SDI
- J2 pad 5: GND -> /MCU/Connectors/VIDEO_OUT
- J3 pad 1: /MCU/Connectors/Mag_SDA -> +5V
- J3 pad 2: /MCU/Connectors/Mag_SCL -> /MCU/Connectors/GPS_RX
- J3 pad 3: +5V -> /MCU/Connectors/GPS_TX
- J3 pad 4: GND -> /MCU/Connectors/I2C_SDA1
- J3 pad 5: /MCU/Connectors/GPS_RX -> /MCU/Connectors/I2C_SCL1
- J3 pad 6: /MCU/Connectors/GPS_TX -> GND
- J7 pad 1: +5V -> GND
- J7 pad 2: GND -> +5V
- R1 pad 1: +3V3 -> +5V
- R1 pad 2: /MCU/Connectors/OSD_VS -> /Peripherals/Power/FB_5V
- R3 pad 1: +3V3 -> /Peripherals/Power/FB_5V
- R3 pad 2: /MCU/Connectors/OSD_LOS -> GND
- R7 pad 1: +5V -> /Peripherals/Power/FB_9V
- R7 pad 2: /Peripherals/Power/FB_5V -> GND
- U1 pad 22: /MCU/Connectors/VTX_TX -> unconnected-(U1-PA0-Pad22)
- U1 pad 23: /MCU/Connectors/VTX_RX -> unconnected-(U1-PA1-Pad23)
- U1 pad 41: unconnected-(U1-PE11-Pad41) -> /MCU/Connectors/OSD_SPI_CS
- U1 pad 42: unconnected-(U1-PE12-Pad42) -> /MCU/Connectors/OSD_SPI_SCK
- U1 pad 43: unconnected-(U1-PE13-Pad43) -> /MCU/Connectors/OSD_SPI_SDO
- U1 pad 44: unconnected-(U1-PE14-Pad44) -> /MCU/Connectors/OSD_SPI_SDI
- U1 pad 59: /MCU/Connectors/Mag_SCL -> /MCU/Connectors/I2C_SCL1
- U1 pad 60: /MCU/Connectors/Mag_SDA -> /MCU/Connectors/I2C_SDA1
- U1 pad 65: /MCU/Connectors/OSD_LOS -> unconnected-(U1-PC8-Pad65)
- U1 pad 66: /MCU/Connectors/OSD_VS -> unconnected-(U1-PC9-Pad66)
- U1 pad 77: unconnected-(U1-PA15-Pad77) -> /MCU/Connectors/BB_SPI_CS
- U1 pad 83: /MCU/Connectors/LPS_SPI_CS -> unconnected-(U1-PD2-Pad83)
- U1 pad 84: /MCU/Connectors/BB_SPI_CS -> unconnected-(U1-PD3-Pad84)
- U1 pad 85: /MCU/Connectors/OSD_SPI_CS -> unconnected-(U1-PD4-Pad85)
Routing:
- net +3V3: track 33.1 -> 104.0 mm
- net /MCU/Connectors/I2C_SCL1: track 0.00 -> 49.3 mm, vias 0 -> 3
- net +5V_USB: track 0.00 -> 43.6 mm, vias 0 -> 3
- net /MCU/Connectors/Mag_SCL: track 42.5 -> 0.00 mm, vias 3 -> 0
- net /MCU/Connectors/I2C_SDA1: track 0.00 -> 42.4 mm, vias 0 -> 4
- net /MCU/Connectors/TELEM_RX: track 24.4 -> 66.3 mm, vias 2 -> 4
- net /MCU/Connectors/Mag_SDA: track 40.5 -> 0.00 mm, vias 3 -> 0
- net /MCU/Connectors/D+: track 1.69 -> 41.2 mm, vias 0 -> 3
- net /MCU/Connectors/D-: track 1.62 -> 41.0 mm, vias 0 -> 2
- net /MCU/Connectors/M4_DSHOT: track 33.9 -> 72.6 mm, vias 3 -> 4
- net /MCU/Connectors/PB10: track 0.00 -> 37.6 mm, vias 0 -> 2
- net /MCU/Connectors/M3_DSHOT: track 34.9 -> 72.0 mm, vias 3 -> 4
- net /MCU/Connectors/ELRS_RX: track 14.1 -> 50.3 mm
- net /MCU/Connectors/M2_DSHOT: track 35.4 -> 71.5 mm, vias 3 -> 4
- net /MCU/Connectors/ELRS_TX: track 16.4 -> 52.4 mm
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- added copper zone on F.Cu, net /MCU/Connectors/NRST
- added copper zone on B.Cu, net GND
- added copper zone on In1.Cu, net GND
- added copper zone on In2.Cu, net GND
- added copper zone on F.Cu, net unconnected-(IC1-~{VSYNC}-Pad17)
- removed copper zone on F.Cu, net /MCU/Connectors/OSD_LOS
- removed copper zone on F.Cu, net /MCU/Connectors/OSD_VS
Other:
- board size 38 x 68 mm -> 39 x 69 mm
