File: Flight_Controller/.history/MCU.kicad_sch (KiCad schematic)
At the start: 38 parts, among them J1 Analog VTX, J10 USB_C_Receptacle_USB2.0_16P, J11 Conn_ARM_SWD_TagConnect_TC203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, J13 SM06B-GHS-TB, J2 Digital VTX, J3 GPS+Mag, J4 ESC Connector, J7 ELRS Reciever, J9 Camera, SW1 SW_Push, U1 STM32H743VITx, U7 TPD2EUSB30ADRTR

Commit message: Almost Done Routing!
Parts:
- added TP1, TP10, TP11, TP12, TP13, TP14, TP15, TP16, TP17, TP18, TP19, TP2, TP20, TP21, TP22, TP23, TP24, TP25, TP3, TP4, TP5, TP6, TP7, TP8, TP9: TestPoint, TestPoint:TestPoint_Pad_D1.0mm, symbol Connector:TestPoint
Connections:
- net +3V3: now also TP3.1
- net +5V: now also TP2.1
- net +5V_USB: now also TP4.1
- net +9V: now also TP1.1
- net +BATT: now also TP5.1
- net ADC_CURR: now also TP16.1
- net D+: now also TP25.1
- net D-: now also TP24.1
- net DVTX_RX: now also TP8.1
- net DVTX_TX: now also TP7.1
- net ELRS_RX: now also TP22.1
- net ELRS_TX: now also TP23.1
- net GND: now also TP6.1
- net GPS_RX: now also TP9.1
- net GPS_TX: now also TP10.1
- net M1_DSHOT: now also TP18.1
- net M2_DSHOT: now also TP19.1
- net M3_DSHOT: now also TP20.1
- net M4_DSHOT: now also TP21.1
- net Mag_SCL: now also TP12.1
- net Mag_SDA: now also TP11.1
- net TELEM_RX: now also TP17.1
- net VIDEO_OUT: now also TP13.1
- net VTX_RX: now also TP14.1
- net VTX_TX: now also TP15.1

Commit message: Routing Done!
Parts:
- removed J1: Analog VTX, Connector_JST:JST_SH_SM05B-SRSS-TB_1x05-1MP_P1.00mm_Horizontal, symbol Connector_Generic:Conn_01x05
- removed TP11, TP12, TP14, TP15: TestPoint, TestPoint:TestPoint_Pad_D1.0mm, symbol Connector:TestPoint
- added R20: 10kΩ, PCM_JLCPCB:R_0603, symbol PCM_JLCPCB-Resistors:0603,10kΩ
- added TP26: TestPoint, TestPoint:TestPoint_Pad_D1.0mm, symbol Connector:TestPoint
Connections:
- net +3V3: now also R20.1
- net +5V: now also J3.1 (Pin_1), J7.2 (Pin_2); no longer J3.3 (Pin_3), J7.1 (Pin_1)
- net BB_SPI_CS: now also U1.77 (PA15); no longer U1.84 (PD3)
- net GND: now also J3.6 (Pin_6), J7.1 (Pin_1); no longer J2.5 (Pin_5), J3.4 (Pin_4), J7.2 (Pin_2)
- net GPS_RX: now also J3.2 (Pin_2); no longer J3.5 (Pin_5)
- net GPS_TX: now also J3.3 (Pin_3); no longer J3.6 (Pin_6)
- net NRST: now also R20.2
- net OSD_SPI_CS: now also U1.41 (PE11); no longer U1.85 (PD4)
- net SBUS: now also TP26.1
- net VIDEO_OUT: now also J2.5 (Pin_5)
- net OSD_SPI_SCK: now reaches U1.42 (PE12)
- net OSD_SPI_SDO: now reaches U1.43 (PE13)
- net OSD_SPI_SDI: now reaches U1.44 (PE14)
- net LPS_SPI_CS: no longer names the net of U1.83 (PD2)
- net Mag_SCL renamed I2C_SCL1
- net I2C_SCL1: now also J3.5 (Pin_5); no longer J3.2 (Pin_2)
- net Mag_SDA renamed I2C_SDA1
- net I2C_SDA1: now also J3.4 (Pin_4); no longer J3.1 (Pin_1)
- net OSD_LOS: no longer names the net of U1.65 (PC8)
- net OSD_VS: no longer names the net of U1.66 (PC9)
- net VTX_RX: no longer names the net of U1.23 (PA1)
- net VTX_TX: no longer names the net of U1.22 (PA0)
- no-connect marks 42 -> 44
Other:
- moved on the sheet: J2, J3, J9, TP13, TP16, TP17, TP18, TP19, TP20
